Commit message: gazebo sim working with robot arm

File: ws/src/robot_arm_ctrl/urdf/robot_arm.xacro (robot description, xacro)
@@ -23,14 +23,4 @@
       hardware_driver="$(arg hardware_driver)"/>
   <xacro:property name="driver" value="$(arg hardware_driver)"/>
-  <!-- Gazebo plugin -->
-  <xacro:if value="${driver == 'gazebo'}">
-    <gazebo reference="world"/>
-    <gazebo>
-      <plugin filename="libgz_ros2_control-system.so" name="gz_ros2_control::GazeboSimROS2ControlPlugin">
-        <parameters>$(arg simulation_controllers)</parameters>
-        <controller_manager_node_name>$(arg prefix)controller_manager</controller_manager_node_name>
-      </plugin>
-    </gazebo>
-  </xacro:if>
   <!-- Webots plugin -->
   <xacro:if value="${driver == 'webots'}">
@@ -39,10 +29,49 @@
     </webots>
   </xacro:if>
-  <!-- Not working at this time -->
-  <gazebo reference="$(arg prefix)shoulder_link">
-    <material>Gazebo/Grey</material>
-    <mu1>0.2</mu1>
-    <mu2>0.2</mu2>
-    <selfCollide>True</selfCollide>
-  </gazebo>
+  <!-- Gazebo plugin -->
+  <xacro:if value="${driver == 'gazebo'}">
+    <gazebo>
+      <plugin filename="gz_ros2_control-system" name="gz_ros2_control::GazeboSimROS2ControlPlugin">
+        <parameters>$(arg simulation_controllers)</parameters>
+      </plugin>
+    </gazebo>
+    <gazebo reference="$(arg prefix)base_link">
+      <material>Gazebo/Orange</material>
+    </gazebo>
+    <gazebo reference="$(arg prefix)shoulder_link">
+      <mu1>0.2</mu1>
+      <mu2>0.2</mu2>
+      <material>Gazebo/Yellow</material>
+    </gazebo>
+    <gazebo reference="$(arg prefix)upper_arm_link">
+      <mu1>0.2</mu1>
+      <mu2>0.2</mu2>
+      <material>Gazebo/Orange</material>
+    </gazebo>
+    <gazebo reference="$(arg prefix)middle_arm_link">
+      <mu1>0.2</mu1>
+      <mu2>0.2</mu2>
+      <material>Gazebo/Orange</material>
+    </gazebo>
+    <gazebo reference="$(arg prefix)fore_arm_link">
+      <mu1>0.2</mu1>
+      <mu2>0.2</mu2>
+      <material>Gazebo/Orange</material>
+    </gazebo>
+    <gazebo reference="$(arg prefix)effector_link">
+      <mu1>0.2</mu1>
+      <mu2>0.2</mu2>
+      <material>Gazebo/Orange</material>
+    </gazebo>
+    <gazebo reference="$(arg prefix)finger_left_link">
+      <mu1>0.2</mu1>
+      <mu2>0.2</mu2>
+      <material>Gazebo/Orange</material>
+    </gazebo>
+    <gazebo reference="$(arg prefix)finger_righ_link">
+      <mu1>0.2</mu1>
+      <mu2>0.2</mu2>
+      <material>Gazebo/Orange</material>
+    </gazebo>
+  </xacro:if>
 </robot>

Commit message: trajectory publisher

File: ws/src/robot_arm_ctrl/urdf/robot_arm.xacro (robot description, xacro)
@@ -37,15 +37,15 @@
     </gazebo>
     <gazebo reference="$(arg prefix)base_link">
-      <material>Gazebo/Orange</material>
+      <material>Gazebo/Gray</material>
     </gazebo>
     <gazebo reference="$(arg prefix)shoulder_link">
       <mu1>0.2</mu1>
       <mu2>0.2</mu2>
-      <material>Gazebo/Yellow</material>
+      <material>Gazebo/Orange</material>
     </gazebo>
     <gazebo reference="$(arg prefix)upper_arm_link">
       <mu1>0.2</mu1>
       <mu2>0.2</mu2>
-      <material>Gazebo/Orange</material>
+      <material>Gazebo/Yellow</material>
     </gazebo>
     <gazebo reference="$(arg prefix)middle_arm_link">
@@ -57,5 +57,5 @@
       <mu1>0.2</mu1>
       <mu2>0.2</mu2>
-      <material>Gazebo/Orange</material>
+      <material>Gazebo/Yellow</material>
     </gazebo>
     <gazebo reference="$(arg prefix)effector_link">
@@ -67,10 +67,10 @@
       <mu1>0.2</mu1>
       <mu2>0.2</mu2>
-      <material>Gazebo/Orange</material>
+      <material>Gazebo/Yellow</material>
     </gazebo>
-    <gazebo reference="$(arg prefix)finger_righ_link">
+    <gazebo reference="$(arg prefix)finger_right_link">
       <mu1>0.2</mu1>
       <mu2>0.2</mu2>
-      <material>Gazebo/Orange</material>
+      <material>Gazebo/Yellow</material>
     </gazebo>
   </xacro:if>
